File: PCB/Using 74HC74N with potentiometer/BSPD.kicad_pcb (KiCad board)
At the start: 2 copper layers, 27 parts, among them U1 sn7476n, U2 LM393, U3 4081, U4 74HC04, U5 LM324, U6 LM324

Commit message: 26.04.2023
Parts:
- R10, R11, R12, R14, R5, R6, R7, R8, R9: footprint Resistor_SMD:R_0201_0603Metric -> Resistor_THT:R_Axial_DIN0204_L3.6mm_D1.6mm_P1.90mm_Vertical
- RV1, RV2: footprint Potentiometer_SMD:Potentiometer_ACP_CA6-VSMD_Vertical -> Potentiometer_THT:Potentiometer_ACP_CA9-H3,8_Horizontal
- moved RV2 25.5 mm to (43.2, 57.1), turned to 90 degrees
- moved R6 23.4 mm to (30.5, 22.9), turned to 180 degrees
- moved R5 18.5 mm to (25.4, 35.6)
- moved TP5 10.2 mm to (71.1, 48.3)
- moved TP4 8.03 mm to (53.3, 58.4)
- moved R11 7.94 mm to (66.0, 58.4)
- moved R7 7.93 mm to (66.0, 55.9)
- moved RV1 7.62 mm to (43.2, 68.6), turned to 90 degrees
- moved TP3 7.62 mm to (22.9, 45.7)
- moved R10 6.98 mm to (40.0, 27.9)
- moved R12 5.83 mm to (60.3, 58.4)
- moved TP1 5.68 mm to (17.8, 45.7)
- moved TP2 5.08 mm to (68.6, 53.3)
- moved U3 5.08 mm to (30.5, 33.0)
- moved U5 5.08 mm to (61.0, 22.9)
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Routing:
- net Net-(R11-Pad1): track 22.8 -> 169.1 mm
- net Net-(R14-Pad2): track 55.8 -> 6.01 mm
- net Net-(U2B--): track 44.1 -> 92.4 mm
- net VCC: track 0.00 -> 43.3 mm
- net Net-(R6-Pad2): track 0.00 -> 20.1 mm
- net Net-(U2B-+): track 13.3 -> 5.08 mm
- net Net-(C1-Pad2): track 68.3 -> 61.8 mm
- net Net-(D2-K): track 58.7 -> 65.2 mm
- net Net-(D1-K): track 43.8 -> 37.6 mm
- net Net-(U6A-+): track 18.6 -> 24.1 mm
- net Net-(U5A-+): track 35.5 -> 31.9 mm
- net Net-(R5-Pad2): track 26.0 -> 23.0 mm
- net Net-(U2A--): track 78.4 -> 76.4 mm
